File: FT2232_JTAG.kicad_sch (KiCad schematic)
At the start: 39 parts, among them J1 USB_C_Receptacle_USB2.0_16P, J2 Conn_01x09, J3 Conn_01x06, U1 FT2232HQ, U2 93LCxxB, U3 MCP1700x-330xxTT, Y1 12.000 MHz

Commit message: wip
Parts:
- added H1, H2, H3, H4: MountingHole, MountingHole:MountingHole_2.2mm_M2_ISO14580, symbol Mechanical:MountingHole
Connections:
- net D+: now reaches J1.A6 (D+), J1.B6 (D+), U1.8 (DP)
- net D-: now reaches J1.A7 (D-), J1.B7 (D-), U1.7 (DM)

Commit message: Fixed pull on BCBUS7
Connections:
- net +3.3VP: now also U1.59 (BCBUS7)
- net GND: now also R11.1
Other:
- moved on the sheet: R11
Changed lines of the file:
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@@
 	)
 	(junction
+		(at 180.34 133.35)
+		(diameter 0)
+		(color 0 0 0 0)
+	)
+	(junction
 		(at 78.74 101.6)
 		(diameter 0)
@@
 	(wire
 		(pts
+			(xy 180.34 133.35) (xy 180.34 135.89)
+		)
+		(stroke
+			(width 0)
+			(type default)
+		)
+	)
+	(wire
+		(pts
 			(xy 59.69 64.77) (xy 57.15 64.77)
 		)
@@
 	(wire
 		(pts
+			(xy 180.34 143.51) (xy 180.34 146.05)
+		)
+		(stroke
+			(width 0)
+			(type default)
+		)
+	)
+	(wire
+		(pts
 			(xy 46.99 72.39) (xy 111.76 72.39)
 		)
@@
 	(wire
 		(pts
-			(xy 184.15 133.35) (xy 187.96 133.35)
-		)
-		(stroke
-			(width 0)
-			(type default)
-		)
-	)
-	(wire
-		(pts
 			(xy 86.36 120.65) (xy 86.36 118.11)
 		)
@@
 	(wire
 		(pts
+			(xy 180.34 133.35) (xy 187.96 133.35)
+		)
+		(stroke
+			(width 0)
+			(type default)
+		)
+	)
+	(wire
+		(pts
 			(xy 243.84 46.99) (xy 243.84 48.26)
 		)
@@
 	(wire
 		(pts
-			(xy 172.72 133.35) (xy 176.53 133.35)
+			(xy 172.72 133.35) (xy 180.34 133.35)
 		)
 		(stroke
@@
 	(symbol
 		(lib_id "Device:R")
-		(at 180.34 133.35 90)
+		(at 180.34 139.7 180)
 		(unit 1)
 		(exclude_from_sim no)
@@
 		(fields_autoplaced yes)
 		(property "Reference" "R11"
-			(at 180.34 127 90)
+			(at 182.88 138.4299 0)
 			(effects
 				(font
 					(size 1.27 1.27)
 				)
+				(justify right)
 			)
 		)
 		(property "Value" "10k"
-			(at 180.34 129.54 90)
+			(at 182.88 140.9699 0)
 			(effects
 				(font
 					(size 1.27 1.27)
 				)
+				(justify right)
 			)
 		)
 		(property "Footprint" "Resistor_SMD:R_0402_1005Metric"
-			(at 180.34 135.128 90)
+			(at 182.118 139.7 90)
 			(effects
 				(font
@@
 		)
 		(property "Datasheet" "~"
-			(at 180.34 133.35 0)
+			(at 180.34 139.7 0)
 			(effects
 				(font
@@
 		)
 		(property "Description" "Resistor"
-			(at 180.34 133.35 0)
+			(at 180.34 139.7 0)
 			(effects
 				(font
@@
 					(unit 1)
 				)
+			)
+		)
+	)
+	(symbol
+		(lib_id "power:GND")
+		(at 180.34 146.05 0)
+		(unit 1)
+		(exclude_from_sim no)
+		(in_bom yes)
+		(on_board yes)
+		(dnp no)
+		(fields_autoplaced yes)
+		(property "Reference" "#PWR036"
+			(at 180.34 152.4 0)
+			(effects
+				(font
+					(size 1.27 1.27)
+				)
+				(hide yes)
+			)
+		)
+		(property "Value" "GND"
+			(at 180.34 151.13 0)
+			(effects
+				(font
+					(size 1.27 1.27)
+				)
+			)
+		)
+		(property "Footprint" ""
+			(at 180.34 146.05 0)
+			(effects
+				(font
+					(size 1.27 1.27)
+				)
+				(hide yes)
+			)
+		)
+		(property "Datasheet" ""
+			(at 180.34 146.05 0)
+			(effects
+				(font
+					(size 1.27 1.27)
+				)
+				(hide yes)
+			)
+		)
+		(property "Description" "Power symbol creates a global label with name \"GND\" , ground"
+			(at 180.34 146.05 0)
+			(effects
+				(font
+					(size 1.27 1.27)
+				)
+				(hide yes)
+			)
+		)
+		(pin "1"
+		)
+		(instances
+			(project "FT2232_JTAG"
+				(path "/a2003e42-1b08-4026-8d40-b256ccd1c2eb"
+					(reference "#PWR036")
+					(unit 1)
+				)

Commit message: added LCSC part numbers
Parts:
- C10, C11, C12, C14, C15, C17, C18, C3, C4, C5, C6, C7, C8, C9: LCSC Part (none) -> C3012376
- C13: LCSC Part (none) -> C695126
- C16, C19: LCSC Part (none) -> C76995
- R1, R11, R2, R3, R5, R6: LCSC Part (none) -> C25531
- R10, R9: LCSC Part (none) -> C25941
- R4: LCSC Part (none) -> C25552
- R7: LCSC Part (none) -> C25752
- R8: LCSC Part (none) -> C102758
- U3: LCSC Part (none) -> C5148688
